Commit message: Updates to URDF

File: acrobot.urdf (robot description, URDF)
Before this commit: robot acrobot, 5 links, 4 joints
Joints:
- joint elbow_joint: limit effort=500 -> lower=-3.14159 upper=3.14159 effort=500

Commit message: First pass at acrobot simulation

File: acrobot.urdf (robot description, URDF)
Before this commit: robot acrobot, 5 links, 4 joints
Joints:
- removed joint planar_x
- removed joint planar_z
- joint planar_roty: parent base_xz -> base

Commit message: remove unused links from URDF

File: acrobot.urdf (robot description, URDF)
Before this commit: robot acrobot, 5 links, 2 joints
Links:
- removed link base_x
- removed link base_xz

Commit message: Correct link masses in URDF, initial version of visualizer

File: acrobot.urdf (robot description, URDF)
Before this commit: robot acrobot, 3 links, 2 joints
Links:
- link blue_link: mass None -> 1
- link red_link: mass None -> 1

Commit message: Add inertia info to URDF

File: acrobot.urdf (robot description, URDF)
Before this commit: robot acrobot, 3 links, 2 joints
Joints:
- joint elbow_joint: type continuous -> revolute

Commit message: Update model of acrobot

File: acrobot.urdf (robot description, URDF)
Before this commit: robot acrobot, 3 links, 2 joints
Joints:
- removed joint planar_roty
- added joint shoulder: type continuous, parent base, child red_link, axis 0 -1 0
